Commit message: rotate optoforce

File: ridgeback_yumi_description/urdf/ridgeback_yumi.urdf (robot description, URDF)
Before this commit: robot ridgeback_yumi, 48 links, 47 joints
Links:
- removed link front_laser
Joints:
- removed joint front_laser_joint
- joint optodaq_r_sensor_link_joint: origin xyz=0 0 -0.033 rpy=3.14159265359 0.0 0.785398163397 -> xyz=0 0 -0.033 rpy=3.14159265359 0.0 0.246898163397
- joint yumi_link_7_r_joint: origin xyz=0 0 0.033 rpy=0 3.14159265359 -0.785398163397 -> xyz=0 0 0.033 rpy=0 3.14159265359 -0.246898163397

File: ridgeback_yumi_description/urdf/ridgeback_yumi.urdf.xacro (robot description, xacro)
@@ -19,5 +19,5 @@
   </xacro:yumi>
   <xacro:yumi_optodaq_sensor name="optodaq_r" parent="yumi_link_7_r">
-      <origin xyz="0 0 0.033" rpy="0 ${PI} ${-PI/4}" />
+      <origin xyz="0 0 0.033" rpy="0 ${PI} ${-PI/4 + 0.5385}" />
   </xacro:yumi_optodaq_sensor>
   <xacro:yumi_optodaq_sensor name="optodaq_l" parent="yumi_link_7_l">
@@ -26,5 +26,5 @@
   <!--right gripper-->
   <xacro:yumi_servo_gripper name="gripper_r" hardware_interface="hardware_interface/EffortJointInterface" parent="optodaq_r_sensor_link">
-    <origin xyz="0 0 -0.033" rpy="${PI} 0.0 ${PI/4}" />
+    <origin xyz="0 0 -0.033" rpy="${PI} 0.0 ${PI/4 + 0.5385}" />
   </xacro:yumi_servo_gripper>
   <!--left gripper-->

Commit message: Current experiment config

File: ridgeback_yumi_description/urdf/ridgeback_yumi.urdf (robot description, URDF)
Before this commit: robot ridgeback_yumi, 47 links, 46 joints
Links:
- added link front_laser, mass 0.130; collision box size=0.05 0.05 0.07; visual mesh filename=package://ridgeback_description/meshes/ust-10lx.stl
- link gripper_l_finger_l: mass 0.01 -> 0.1
- link gripper_l_finger_r: mass 0.01 -> 0.1
- link gripper_r_finger_l: mass 0.01 -> 0.1
- link gripper_r_finger_r: mass 0.01 -> 0.1
Joints:
- removed joint optodaq_l_sensor_link_joint
- removed joint optodaq_r_sensor_link_joint
- added joint front_laser_joint: type fixed, parent chassis_link, child front_laser, origin xyz=0.3932 0 0.2330 rpy=0 0 0.0
- added joint yumi_link_7_l_joint_daq: type fixed, parent yumi_link_7_l, child optodaq_l_sensor_link, origin xyz=0 0 0.033 rpy=0 3.14159265359 -0.3
- added joint yumi_link_7_r_joint_daq: type fixed, parent yumi_link_7_r, child optodaq_r_sensor_link, origin xyz=0 0 0.033 rpy=0 3.14159265359 -0.3
- joint yumi_link_7_l_joint: child optodaq_l_sensor_link -> gripper_l_base; origin xyz=0 0 0.033 rpy=0 3.14159265359 -0.785398163397 -> xyz=0 0 0.066 rpy=0.0 0.0 1.57079632679
- joint yumi_link_7_r_joint: child optodaq_r_sensor_link -> gripper_r_base; origin xyz=0 0 0.033 rpy=0 3.14159265359 -0.246898163397 -> xyz=0 0 0.066 rpy=0.0 0.0 1.57079632679

File: ridgeback_yumi_description/urdf/ridgeback_yumi.urdf.xacro (robot description, xacro)
@@ -19,16 +19,16 @@
   </xacro:yumi>
   <xacro:yumi_optodaq_sensor name="optodaq_r" parent="yumi_link_7_r">
-      <origin xyz="0 0 0.033" rpy="0 ${PI} ${-PI/4 + 0.5385}" />
+      <origin xyz="0 0 0.033" rpy="0 ${PI} -0.3" />
   </xacro:yumi_optodaq_sensor>
   <xacro:yumi_optodaq_sensor name="optodaq_l" parent="yumi_link_7_l">
-	  <origin xyz="0 0 0.033" rpy="0 ${PI} ${-PI/4}" />
+	  <origin xyz="0 0 0.033" rpy="0 ${PI} -0.3" />
   </xacro:yumi_optodaq_sensor>
   <!--right gripper-->
-  <xacro:yumi_servo_gripper name="gripper_r" hardware_interface="hardware_interface/EffortJointInterface" parent="optodaq_r_sensor_link">
-    <origin xyz="0 0 -0.033" rpy="${PI} 0.0 ${PI/4 + 0.5385}" />
+  <xacro:yumi_servo_gripper name="gripper_r" hardware_interface="hardware_interface/EffortJointInterface" parent="yumi_link_7_r">
+    <origin xyz="0 0 0.066" rpy="0.0 0.0 ${PI/2}" />
   </xacro:yumi_servo_gripper>
   <!--left gripper-->
-  <xacro:yumi_servo_gripper name="gripper_l" hardware_interface="hardware_interface/EffortJointInterface" parent="optodaq_l_sensor_link">
-    <origin xyz="0 0 -0.033" rpy="${PI} 0.0 ${PI/4}" />
+  <xacro:yumi_servo_gripper name="gripper_l" hardware_interface="hardware_interface/EffortJointInterface" parent="yumi_link_7_l">
+    <origin xyz="0 0 0.066" rpy="0.0 0.0 ${PI/2}" />
   </xacro:yumi_servo_gripper>
   <xacro:property name="pedestal_height" value="0.28" />

Commit message: Current calibration files

File: ridgeback_yumi_description/urdf/ridgeback_yumi.urdf (robot description, URDF)
Before this commit: robot ridgeback_yumi, 48 links, 47 joints
Links:
- added link fold_case_object_link; visual cylinder length=0.24 radius=0.06
- added link rod_piece_object_link; visual cylinder length=0.16 radius=0.06
Joints:
- added joint gripper_l_base_joint_rod: type fixed, parent gripper_l_base, child rod_piece_object_link, origin xyz=0 0 0.17 rpy=0 0 0
- added joint gripper_r_base_joint_fold: type fixed, parent gripper_r_base, child fold_case_object_link, origin xyz=0 0 0.21 rpy=0 0 0

File: ridgeback_yumi_description/urdf/ridgeback_yumi.urdf.xacro (robot description, xacro)
@@ -12,4 +12,7 @@
   <!--Import the yumi optodaq sensors macro -->
   <xacro:include filename="$(find yumi_description)/urdf/Extras/yumi_optodaq_sensors.xacro"/>
+  <!--Import folding macros -->
+  <xacro:include filename="$(find yumi_description)/urdf/Extras/yumi_fold_case.xacro"/>
+  <xacro:include filename="$(find yumi_description)/urdf/Extras/yumi_rod.xacro"/>
   <!-- Import Gazebo plugins -->
   <xacro:include filename="$(find yumi_description)/urdf/Gazebo/gazebo.urdf.xacro"/>
@@ -32,4 +35,12 @@
     <origin xyz="0 0 0.066" rpy="0.0 0.0 ${PI/2}" />
   </xacro:yumi_servo_gripper>
+  <!-- Surface piece -->
+ <xacro:yumi_fold_case name="fold_case" parent="gripper_r_base">
+   <origin xyz="0 0 0.21" rpy="0 0 0" />
+ </xacro:yumi_fold_case>
+ <!-- Rod piece -->
+ <xacro:yumi_rod name="rod_piece" parent="gripper_l_base">
+   <origin xyz="0 0 0.17" rpy="0 0 0" />
+ </xacro:yumi_rod>
   <xacro:property name="pedestal_height" value="0.28" />
   <xacro:property name="pedestal_offset_x" value="0.32" />
