Commit message: Integration of spinning_lidar URDF and launch commands

File: ridgeback_yumi_description/urdf/ridgeback_yumi.urdf.xacro (robot description, xacro)
@@ -14,4 +14,6 @@
   <!-- Import Gazebo plugins -->
   <xacro:include filename="$(find yumi_description)/urdf/Gazebo/gazebo.urdf.xacro"/>
+  <!-- Import spinning_lidar macro and Gazebo plugins -->
+  <xacro:include filename="$(find spinning_lidar_description)/urdf/rotating_mounts/rotating_mount_v1.urdf.xacro" />
   <!--yumi-->
   <xacro:yumi name="yumi" hardware_interface="hardware_interface/VelocityJointInterface" parent="yumi_pedestal">
@@ -35,7 +37,5 @@
   <xacro:property name="pedestal_offset_x" value="0.32" />
   <xacro:property name="yumi_offset_x" value="0.06" />
-  <xacro:property name="yumi_height" value="0.25" />
-  <xacro:property name="kinect_zrotation_fix" value="${- PI / 2.0}" />
-  <xacro:property name="kinect_base_pitch" value="${ -PI/2.0 }" />
+  <xacro:property name="yumi_offset_z" value="0.25" />
   <joint name="ridgeback_base_to_pedestal" type="fixed">
     <origin rpy="0 0 ${PI}" xyz="${pedestal_offset_x} 0 ${pedestal_height}" />
@@ -60,63 +60,14 @@
   </link>
   <joint name="pedestal_to_yumi" type="fixed">
-    <origin rpy="0 0 ${PI}" xyz="${yumi_offset_x} 0 ${yumi_height}" />
+    <origin rpy="0 0 ${PI}" xyz="${yumi_offset_x} 0 ${yumi_offset_z}" />
+    <axis xyz="0 0 0"/>
     <parent link="yumi_pedestal" />
     <child link="yumi_base_link" />
   </joint>
-  <link name="kinect2">
-    <visual>
-      <origin xyz="0 0 0" rpy="0 0 0" />
-      <geometry>
-        <mesh scale="0.001 0.001 0.001" filename="package://yumi_description/meshes/accesories/KinectXboxOne.stl"/>
-      </geometry>
-      <material name="Black" />
-    </visual>
-  </link>
-  <link name="left_kinect_base">
-      <visual>
-        <origin xyz="0 0 0" rpy="0 0 0" />
-        <geometry>
-          <box size="0.4 0.02 0.02" />
-        </geometry>
-        <material name="Grey" />
-      </visual>
-  </link>
-  <link name="right_kinect_base">
-      <visual>
-        <origin xyz="0 0 0" rpy="0 0 0" />
-        <geometry>
-          <box size="0.4 0.02 0.02" />
-        </geometry>
-        <material name="Grey" />
-      </visual>
-  </link>
-  <link name="middle_kinect_base">
-      <visual>
-        <origin xyz="0 0 0" rpy="0 0 0" />
-        <geometry>
-          <box size="0.4 0.02 0.02" />
-        </geometry>
-        <material name="Grey" />
-      </visual>
-  </link>
-   <joint name="kinect2_to_right_kinect_base" type="fixed">
-    <parent link="yumi_base_link" />
-    <child link="right_kinect_base" />
-    <origin rpy="0 ${-PI/2} 0.17" xyz="-0.1 -0.03 0.56" />
-  </joint>
-  <joint name="kinect2_to_left_kinect_base" type="fixed">
-    <parent link="yumi_base_link" />
-    <child link="left_kinect_base" />
-    <origin rpy="0 ${-PI/2} -0.17" xyz="-0.1 0.03 0.56" />
-  </joint>
-  <joint name="yumi_to_middle_kinect_base" type="fixed">
-    <parent link="yumi_base_link" />
-    <child link="middle_kinect_base" />
-    <origin rpy="0 ${kinect_base_pitch} 0" xyz="-0.1 0 0.56" />
-  </joint>
-  <joint name="middle_kinect_base_to_kinect2" type="fixed">
-    <parent link="middle_kinect_base" />
-    <child link="kinect2" />
-    <origin rpy="${-PI/2} 0 ${kinect_zrotation_fix}" xyz="0.25 0 0" />
-  </joint>
+  <xacro:property name="yumi_height" value="0.465" />
+  <xacro:property name="spinning_lidar_x_offset" value="-0.15" />
+  <xacro:property name="spinning_lidar_y_offset" value="0" />
+  <xacro:rotating_mount_v1_macro parent="yumi_base_link" mount_link="laser_mount" axis_link="laser_axis" lidar_link="laser">
+      <origin rpy="0 0 ${PI}" xyz="${spinning_lidar_x_offset} ${spinning_lidar_y_offset} ${yumi_height}" />
+  </xacro:rotating_mount_v1_macro>
 </robot>

Commit message: Update transforms for incorrectly mounted FT sensors

File: ridgeback_yumi_description/urdf/ridgeback_yumi.urdf.xacro (robot description, xacro)
@@ -19,16 +19,16 @@
   </xacro:yumi>
   <xacro:yumi_optodaq_sensor name="optodaq_r" parent="yumi_link_7_r">
-      <origin xyz="0 0 0.033" rpy="0 ${PI} -0.3" />
+      <origin xyz="0 0 0.033" rpy="0 ${PI} 3.67" />
   </xacro:yumi_optodaq_sensor>
   <xacro:yumi_optodaq_sensor name="optodaq_l" parent="yumi_link_7_l">
-	  <origin xyz="0 0 0.033" rpy="0 ${PI} -0.3" />
+	  <origin xyz="0 0 0.033" rpy="0 ${PI} -1.9" />
   </xacro:yumi_optodaq_sensor>
   <!--right gripper-->
   <xacro:yumi_servo_gripper name="gripper_r" hardware_interface="hardware_interface/EffortJointInterface" parent="yumi_link_7_r">
-    <origin xyz="0 0 0.066" rpy="0.0 0.0 ${PI/2}" />
+    <origin xyz="0 0 0.066" rpy="0.0 0.0 -3.948" />
   </xacro:yumi_servo_gripper>
   <!--left gripper-->
   <xacro:yumi_servo_gripper name="gripper_l" hardware_interface="hardware_interface/EffortJointInterface" parent="yumi_link_7_l">
-    <origin xyz="0 0 0.066" rpy="0.0 0.0 ${PI/2}" />
+    <origin xyz="0 0 0.066" rpy="0.0 0.0 0.818" />
   </xacro:yumi_servo_gripper>
   <xacro:property name="pedestal_height" value="0.28" />
